File: NFC_harvester_battery_free/hardware/Densor_kicad_project/densor_nfc_v2.kicad_sch (KiCad schematic)
At the start: 26 parts, among them J1 Conn_ARM_JTAG_SWD_10, J2 Conn_01x08_Pin, J3 Conn_01x04_Pin, U1 ST25DV04K-JFR6D3, U2 AM1805, U3 MAX30208CLB+, U4 STM32L011F3Ux, U5 LIS2DW12, U6 TS3A44159, Y1 Crystal

Commit message: Schemetics and PCB layout finished
Concept diagram added
Changed lines of the file:
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@@
 	)
 	(no_connect
+		(at 204.47 107.95)
+	)
+	(no_connect
 		(at 50.8 55.88)
 	)
@@
 	)
 	(no_connect
-		(at 204.47 107.95)
-	)
-	(no_connect
 		(at 96.52 158.75)
 	)
@@
 	)
 	(no_connect
-		(at 204.47 100.33)
-	)
-	(no_connect
 		(at 119.38 148.59)
 	)
@@
 	)
 	(no_connect
+		(at 204.47 100.33)
+	)
+	(no_connect
 		(at 53.34 166.37)
 	)
@@
 	(wire
 		(pts
-			(xy 207.01 102.87) (xy 204.47 102.87)
-		)
-		(stroke
-			(width 0)
-			(type default)
-		)
-	)
-	(wire
-		(pts
 			(xy 194.31 160.02) (xy 204.47 160.02)
 		)
@@
 	(wire
 		(pts
+			(xy 204.47 102.87) (xy 207.01 102.87)
+		)
+		(stroke
+			(width 0)
+			(type default)
+		)
+	)
+	(wire
+		(pts
 			(xy 209.55 68.58) (xy 209.55 73.66)
 		)
@@
 			)
 		)
-		(property "Datasheet" "MAX30208CLB+"
+		(property "Datasheet" "https://www.analog.com/media/en/technical-documentation/data-sheets/MAX30208.pdf"
 			(at 163.83 100.33 0)
 			(hide yes)
